File: pcb/kicad/pcb.kicad_pcb (KiCad board)
At the start: 2 copper layers, 226 parts, among them J1 MX-NoLED, K0 MX-NoLED, K1 MX-NoLED, K10 MX-NoLED, K2 MX-NoLED, K3 MX-NoLED, K4 MX-NoLED, K5 MX-NoLED, K6 MX-NoLED, K7 MX-NoLED, K8 MX-NoLED, K9 MX-NoLED, M1 MX-NoLED, P1 MX-NoLED, Q1 MX-NoLED, SW1 SW_Push, T1 MX-NoLED, U1 MX-NoLED, U2 AT90USB1286-AU, X1 MX-NoLED, Y1 MX-NoLED, Y2 16 MHz

Commit message: pcb: move diodes next to switches
Parts:
- D1, D10, D100, D101, D102, D103, D104, D105, D106, D11, D12, D13, D14, D15, D16, D17, D18, D19, D2, D20, D21, D22, D23, D24, D25, D26, D27, D28, D29, D3, D30, D31, D32, D33, D34, D35, D36, D37, D38, D39, D4, D40, D41, D42, D43, D44, D45, D46, D47, D48, D49, D5, D50, D51, D52, D53, D54, D55, D56, D57, D58, D6, D60, D61, D62, D63, D64, D65, D66, D67, D68, D69, D7, D70, D71, D72, D73, D74, D75, D76, D77, D78, D79, D8, D80, D81, D82, D83, D84, D85, D86, D87, D88, D89, D9, D90, D91, D92, D93, D94, D95, D96, D97, D98, D99: moved to B.Cu
- moved D75 444.5 mm to (415.2, -48.3), turned to 90 degrees
- moved D58 435.4 mm to (433.4, -67.0), turned to 270 degrees
- moved D57 422.6 mm to (415.2, -67.3), turned to 90 degrees
- moved D56 415.9 mm to (396.1, -67.3), turned to 90 degrees
- moved D74 403.7 mm to (396.4, -48.0), turned to 90 degrees
- moved D73 401.2 mm to (377.0, -48.3), turned to 90 degrees
- moved D93 397.0 mm to (433.2, -28.9), turned to 270 degrees
- moved D36 390.6 mm to (415.0, -86.4), turned to 90 degrees
- moved D92 388.6 mm to (415.1, -29.2), turned to 90 degrees
- moved D55 385.8 mm to (377.1, -67.4), turned to 90 degrees
- moved D16 379.8 mm to (353.5, -115.0), turned to 90 degrees
- moved D53 373.1 mm to (334.3, -67.3), turned to 90 degrees
- moved D37 372.3 mm to (433.7, -86.4), turned to 90 degrees
- moved D54 367.9 mm to (353.3, -67.3), turned to 90 degrees
- moved D15 364.7 mm to (334.1, -114.9), turned to 90 degrees
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
Commit message: pcb: position components
Parts:
- C2, C3, C4, C5, C6, C7, C8, F14, R2, R3, R4, R5, SW1, U2, USB1, Y2: moved to B.Cu
- moved F14 346.0 mm to (-27.8, 38.5), turned to 90 degrees
- moved R4 341.0 mm to (-23.6, 38.5), turned to 90 degrees
- moved R3 339.8 mm to (-20.1, 38.6), turned to 90 degrees
- moved SW1 214.8 mm to (254.9, 103.9), turned to 90 degrees
- moved D105 160.4 mm to (328.0, 133.5), turned to 270 degrees
- moved D14 160.1 mm to (256.3, 33.9)
- moved D16 160.1 mm to (294.5, 33.9)
- moved D31 160.1 mm to (256.3, 62.3)
- moved D32 160.1 mm to (275.3, 62.3)
- moved D33 160.1 mm to (294.1, 62.5)
- moved D35 160.1 mm to (337.4, 62.5)
- moved D50 160.1 mm to (203.8, 81.5)
- moved D53 160.1 mm to (275.3, 81.5)
- moved D54 160.1 mm to (294.3, 81.5)
- moved D74 160.1 mm to (337.4, 100.8)
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Connections:
- U2 pad 12: COL11 -> Net-(U2-Pad12)
- U2 pad 13: COL10 -> Net-(U2-Pad13)
- U2 pad 14: COL9 -> Net-(U2-Pad14)
- U2 pad 15: COL8 -> Net-(U2-Pad15)
- U2 pad 16: COL7 -> Net-(U2-Pad16)
- U2 pad 17: COL6 -> Net-(U2-Pad17)
- U2 pad 27: ROW5 -> Net-(U2-Pad27)
- U2 pad 28: ROW4 -> Net-(U2-Pad28)
- U2 pad 29: ROW3 -> Net-(U2-Pad29)
- U2 pad 30: ROW2 -> Net-(U2-Pad30)
- U2 pad 31: ROW1 -> Net-(U2-Pad31)
- U2 pad 32: ROW0 -> Net-(U2-Pad32)
- U2 pad 37: COL5 -> Net-(U2-Pad37)
- U2 pad 38: COL4 -> Net-(U2-Pad38)
- U2 pad 39: COL3 -> Net-(U2-Pad39)
- U2 pad 40: COL2 -> Net-(U2-Pad40)
- U2 pad 41: COL1 -> Net-(U2-Pad41)
- U2 pad 42: COL0 -> Net-(U2-Pad42)
- U2 pad 44: COL12 -> Net-(U2-Pad44)
- U2 pad 45: COL13 -> Net-(U2-Pad45)
- U2 pad 46: COL14 -> Net-(U2-Pad46)
- U2 pad 47: COL15 -> Net-(U2-Pad47)
- U2 pad 48: COL16 -> Net-(U2-Pad48)
- U2 pad 49: COL17 -> Net-(U2-Pad49)
- U2 pad 54: COL18 -> Net-(U2-Pad54)
- U2 pad 55: COL19 -> Net-(U2-Pad55)
- U2 pad 56: COL20 -> Net-(U2-Pad56)
- U2 pad 57: COL21 -> Net-(U2-Pad57)
Other:
- board outline added: 431.8 x 127 mm

Commit message: pcb: finish mcu positioning
Parts:
- moved C5 111.0 mm to (319.2, 51.4), turned to 180 degrees
- moved R5 107.1 mm to (326.5, 44.3)
- moved U2 104.2 mm to (316.0, 41.3)
- moved C6 103.4 mm to (305.3, 42.3), turned to 270 degrees
- moved C4 103.2 mm to (307.6, 30.0)
- moved C3 103.0 mm to (311.1, 28.8), turned to 90 degrees
- moved C2 102.9 mm to (319.7, 28.8)
- moved C7 102.8 mm to (304.7, 49.1), turned to 270 degrees
- moved Y2 102.7 mm to (315.5, 29.2), turned to 225 degrees
- moved C8 101.0 mm to (302.0, 43.3)
- moved R2 98.6 mm to (299.3, 31.2), turned to 180 degrees
- moved SW1 81.0 mm to (300.4, 36.8), turned to 270 degrees
- moved USB1 2.01 mm to (-22.9, 29.8)
- moved F14 1.82 mm to (-26.0, 38.9)
- moved R3 1.65 mm to (-21.6, 39.2)
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Connections:
- U2 pad 10: Net-(U2-Pad10) -> COL16
- U2 pad 11: Net-(U2-Pad11) -> COL15
- U2 pad 12: Net-(U2-Pad12) -> COL14
- U2 pad 13: Net-(U2-Pad13) -> COL13
- U2 pad 14: Net-(U2-Pad14) -> COL12
- U2 pad 15: Net-(U2-Pad15) -> COL11
- U2 pad 17: Net-(U2-Pad17) -> ROW0
- U2 pad 54: Net-(U2-Pad54) -> COL7
- U2 pad 55: Net-(U2-Pad55) -> COL6
- U2 pad 56: Net-(U2-Pad56) -> COL5
- U2 pad 57: Net-(U2-Pad57) -> COL4
- U2 pad 58: Net-(U2-Pad58) -> COL3
- U2 pad 59: Net-(U2-Pad59) -> COL2
- U2 pad 60: Net-(U2-Pad60) -> COL1
- U2 pad 61: Net-(U2-Pad61) -> COL0
- U2 pad 9: Net-(U2-Pad9) -> COL17
Routing:
- net ROW1: track 0.00 -> 587.1 mm
- net ROW2: track 0.00 -> 534.2 mm
- net ROW4: track 0.00 -> 515.3 mm
- net ROW3: track 0.00 -> 488.0 mm
- net ROW5: track 0.00 -> 482.3 mm
- net ROW0: track 0.00 -> 480.5 mm, vias 0 -> 2
- net GND: track 0.00 -> 422.5 mm
- net +5V: track 0.00 -> 409.4 mm, vias 0 -> 4
- net Net-(R4-Pad1): track 0.00 -> 335.7 mm
- net Net-(R3-Pad1): track 0.00 -> 333.8 mm
- net COL11: track 0.00 -> 270.6 mm, vias 0 -> 1
- net COL13: track 0.00 -> 235.2 mm, vias 0 -> 1
- net COL14: track 0.00 -> 222.2 mm, vias 0 -> 1
- net COL12: track 0.00 -> 209.5 mm, vias 0 -> 1
- net COL15: track 0.00 -> 179.4 mm, vias 0 -> 1
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Other:
- net class Default: trace_width 0.25 -> 0.254
- net class Power added: clearance 0.2, trace_width 0.381, via_dia 0.8, via_drill 0.4

Commit message: pcb: finish tracks on pcb
Parts:
- moved USB1 2.04 mm to (-23.0, 27.8)
- moved Y2 0.51 mm to (315.5, 29.7)
Connections:
- U2 pad 34: Net-(U2-Pad34) -> COL21
- U2 pad 35: Net-(U2-Pad35) -> COL20
- U2 pad 36: Net-(U2-Pad36) -> COL19
- U2 pad 37: Net-(U2-Pad37) -> COL18
- U2 pad 38: Net-(U2-Pad38) -> ROW1
- U2 pad 39: Net-(U2-Pad39) -> ROW2
- U2 pad 40: Net-(U2-Pad40) -> ROW3
- U2 pad 41: Net-(U2-Pad41) -> ROW4
- U2 pad 42: Net-(U2-Pad42) -> ROW5
- U2 pad 49: Net-(U2-Pad49) -> COL10
- U2 pad 50: Net-(U2-Pad50) -> COL9
- U2 pad 51: Net-(U2-Pad51) -> COL8
Routing:
- net COL0: track 108.0 -> 476.1 mm
- net COL1: track 79.1 -> 429.0 mm
- net COL2: track 96.9 -> 428.3 mm
- net COL3: track 121.2 -> 434.5 mm
- net COL4: track 96.8 -> 391.7 mm
- net COL5: track 96.7 -> 373.4 mm
- net COL6: track 87.5 -> 346.1 mm
- net COL7: track 100.2 -> 340.4 mm
- net COL8: track 100.1 -> 329.1 mm
- net COL9: track 100.1 -> 311.1 mm
- net COL10: track 119.2 -> 311.1 mm
- net ROW5: track 482.3 -> 617.7 mm, vias 0 -> 2
- net ROW4: track 515.3 -> 633.4 mm, vias 0 -> 2
- net ROW3: track 488.0 -> 591.7 mm, vias 0 -> 2
- net ROW2: track 534.2 -> 614.6 mm, vias 0 -> 2
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- added copper zone on B.Cu, net GND
Other:
- board text removed: "rs"
