File: pcb/pcb.sch (KiCad schematic (older format))
At the start: 226 parts, among them J1 MX-NoLED, K0 MX-NoLED, K1 MX-NoLED, K10 MX-NoLED, K2 MX-NoLED, K3 MX-NoLED, K4 MX-NoLED, K5 MX-NoLED, K6 MX-NoLED, K7 MX-NoLED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

Commit message: pcb: improve board design
Parts:
- removed F14: 500mA, Fuse:Fuse_1206_3216Metric, symbol Device:Polyfuse_Small
- added FB1: Ferrite_Bead_Small, Resistor_SMD:R_0805_2012Metric, symbol Device:Ferrite_Bead_Small
- added LED_CPSLK1, LED_NUMLK1: LED_Small, LED_SMD:LED_0805_2012Metric, symbol Device:LED_Small
- added R10, R11, R12, R13, R7, R9: 10K, Resistor_SMD:R_0805_2012Metric, symbol Device:R_Small
- added R_CPSLK1, R_NUMLK1: 90, Resistor_SMD:R_0805_2012Metric, symbol Device:R_Small
- added U3: EMI2121MTTAG, Package_DFN_QFN:WDFN-8-1EP_2x2.2mm_P0.5mm_EP0.80x0.54, symbol Power_Protection:EMI2121MTTAG
- BKSP1, ENTER1, NP-0, NP-ENTER1, NP-PLUS1: footprint MX_Alps_Hybrid:MX-1U-NoLED -> MX_Alps_Hybrid:MX-2U-NoLED
- MX-RSHIFT1: footprint MX_Alps_Hybrid:MX-1U-NoLED -> MX_Alps_Hybrid:MX-2.75U-NoLED
- SPACE1: footprint MX_Alps_Hybrid:MX-1U-NoLED -> MX_Alps_Hybrid:MX-6.25U-NoLED
Connections:
- net +5V: now also FB1.1, R10.2, R11.2, R12.2, R13.2, R7.2, R9.2, R_CPSLK1.1, R_NUMLK1.1
- net D+: now also U3.8 (Out_1+); no longer USB1.3 (D+)
- net D-: now also U3.7 (Out_1-); no longer USB1.4 (D-)
- net GND: now also USB1.6 (SHIELD), U3.3 (GND), U3.4 (GND), U3.5 (GND), U3.9 (GND)
- net ROW0: now also R7.1
- net ROW5: now also R13.1
- net VCC: now also FB1.2, U3.6 (VDD)
- net NUMLKLED: now reaches U2.32 (PD7)
- net NUMLKLED: now also LED_NUMLK1.1 (K)
- net CPSLKLED: now reaches U2.33 (PE0)
- net CPSLKLED: now also LED_CPSLK1.1 (K)
- new net: U3.1 (In_1+), USB1.3 (D+)
- new net: U3.2 (In_1-), USB1.4 (D-)
- new net: LED_CPSLK1.2 (A), R_CPSLK1.2
- new net: LED_NUMLK1.2 (A), R_NUMLK1.2
Other:
- moved on the sheet: C4, C5, C6, C7, USB1

Commit message: pcb: change to usb-c, reorganise pcb
Parts:
- removed R10, R11, R12, R13, R7: 10K, Resistor_SMD:R_0805_2012Metric, symbol Device:R_Small
- removed U3: EMI2121MTTAG, Package_DFN_QFN:WDFN-8-1EP_2x2.2mm_P0.5mm_EP0.80x0.54, symbol Power_Protection:EMI2121MTTAG
- removed USB1: Molex-0548190589, random-keyboard-parts:Molex-0548190589, symbol random-keyboard-parts:Molex-0548190589
- added C9: 0.1uF, Capacitor_SMD:C_0805_2012Metric, symbol Device:C_Small
- added F14: 500mA, Fuse:Fuse_0805_2012Metric, symbol Device:Polyfuse_Small
- added J2: AVR-ISP-6, random-keyboard-parts:Reset_Pretty-Mask, symbol Connector:AVR-ISP-6
- added R8: 5.1k, Resistor_SMD:R_0805_2012Metric, symbol Device:R_Small
- added U3: PRTR5V0U2X, random-keyboard-parts:SOT143B, symbol random-keyboard-parts:PRTR5V0U2X
- added USB1: HRO-TYPE-C-31-M-12, Type-C:HRO-TYPE-C-31-M-12, symbol Type-C:HRO-TYPE-C-31-M-12
- A1: value MX-NoLED -> A
- ALT1, RALT1: value MX-NoLED -> Alt
- AT1: value MX-NoLED -> @
- B1: value MX-NoLED -> B
- BKSP1: value MX-NoLED -> Backspace
- BSLSH1: value MX-NoLED -> \\
- C1: value MX-NoLED -> C
- CAPSL1: value MX-NoLED -> Caps Lock
- COLON1: value MX-NoLED -> :
- COMMA1: value MX-NoLED -> ,
- CTRL1, RCTRL1: value MX-NoLED -> Ctrl
- D59: value MX-NoLED -> D
- DARROW1: value MX-NoLED -> Down
- DASH1, NP-MINUS1: value MX-NoLED -> -
- DEL1, NP-DEL1: value MX-NoLED -> Del
- E1: value MX-NoLED -> E
- END1: value MX-NoLED -> End
- ENTER1, NP-ENTER1: value MX-NoLED -> Enter
- EQUALS1: value MX-NoLED -> =
- ESC1: value MX-NoLED -> Esc
- F1: value MX-NoLED -> F1
- F10: value MX-NoLED -> F10
- F11: value MX-NoLED -> F11
- F12: value MX-NoLED -> F12
- F13: value MX-NoLED -> F
- F2: value MX-NoLED -> F2
- F3: value MX-NoLED -> F3
- F4: value MX-NoLED -> F4
- F5: value MX-NoLED -> F5
- F6: value MX-NoLED -> F6
- F7: value MX-NoLED -> F7
- F8: value MX-NoLED -> F8
- F9: value MX-NoLED -> F9
- FB1: value Ferrite_Bead_Small -> 500mA
- FSLSH1, NP-DIV1: value MX-NoLED -> /
- G1: value MX-NoLED -> G
- H1: value MX-NoLED -> H
- HASH1: value MX-NoLED -> #
- HOME1: value MX-NoLED -> Home
- I1: value MX-NoLED -> I
- INS1: value MX-NoLED -> Insert
- J1: value MX-NoLED -> J
- K0, NP-0: value MX-NoLED -> 0
- K1, NP-1: value MX-NoLED -> 1
- K10: value MX-NoLED -> K
- K2, NP-2: value MX-NoLED -> 2
- K3, NP-3: value MX-NoLED -> 3
- K4, NP-4: value MX-NoLED -> 4
- K5, NP-5: value MX-NoLED -> 5
- K6, NP-6: value MX-NoLED -> 6
- K7, NP-7: value MX-NoLED -> 7
- K8, NP-8: value MX-NoLED -> 8
- K9, NP-9: value MX-NoLED -> 9
- L1: value MX-NoLED -> L
- LARROW1: value MX-NoLED -> Left
- LCBR1: value MX-NoLED -> {
- M1: value MX-NoLED -> M
- MENU1: value MX-NoLED -> Menu
- MX-RSHIFT1, SHIFT1: value MX-NoLED -> Shift
- N1: value MX-NoLED -> N
- NP-MTPLY1: value MX-NoLED -> *
- NP-PLUS1: value MX-NoLED -> +
- NUMLK1: value MX-NoLED -> Num Lock
- O1: value MX-NoLED -> O
- P1: value MX-NoLED -> P
- PAUSE1: value MX-NoLED -> Pause
- PERIOD1: value MX-NoLED -> .
- PGDN1: value MX-NoLED -> Page Down
- PGUP1: value MX-NoLED -> Page Up
- PRTSC1: value MX-NoLED -> Print Screen
- Q1: value MX-NoLED -> Q
- R1: value MX-NoLED -> R
- R9: value 10K -> 5.1k
- RARROW1: value MX-NoLED -> Right
- RCBR1: value MX-NoLED -> }
- S1: value MX-NoLED -> S
- SCLLK1: value MX-NoLED -> Scroll Lock
- SPACE1: value MX-NoLED -> Space
- T1: value MX-NoLED -> T
- TAB1: value MX-NoLED -> Tab
- TILDA1: value MX-NoLED -> ~
- U1: value MX-NoLED -> U
- UARROW1: value MX-NoLED -> Up
- V1: value MX-NoLED -> V
- W1: value MX-NoLED -> W
- WIN1, WIN2: value MX-NoLED -> Win
- X1: value MX-NoLED -> X
- Y1: value MX-NoLED -> Y
- Z1: value MX-NoLED -> Z
Connections:
- net +5V: now also C9.1, J2.2 (VCC); no longer R9.2
- net COL1: now also U2.33 (PE0); no longer U2.60 (PF1)
- net COL10: now also U2.42 (PC7); no longer U2.49 (PA2)
- net COL11: now also U2.45 (PA6); no longer U2.15 (PB5)
- net COL12: now also U2.46 (PA5); no longer U2.14 (PB4)
- net COL13: now also U2.47 (PA4); no longer U2.13 (PB3)
- net COL14: now also U2.48 (PA3); no longer U2.12 (PB2)
- net COL15: now also U2.15 (PB5); no longer U2.11 (PB1)
- net COL16: now also U2.16 (PB6); no longer U2.10 (PB0)
- net COL17: now also U2.17 (PB7); no longer U2.9 (PE3)
- net COL18: now also U2.31 (PD6); no longer U2.37 (PC2)
- net COL19: now also U2.30 (PD5); no longer U2.36 (PC1)
- net COL2: now also U2.34 (PE1); no longer U2.59 (PF2)
- net COL20: now also U2.29 (PD4); no longer U2.35 (PC0)
- net COL21: now also U2.28 (PD3); no longer U2.34 (PE1)
- net COL3: now also U2.35 (PC0); no longer U2.58 (PF3)
- net COL4: now also U2.36 (PC1); no longer U2.57 (PF4)
- net COL5: now also U2.37 (PC2); no longer U2.56 (PF5)
- net COL6: now also U2.38 (PC3); no longer U2.55 (PF6)
- net COL7: now also U2.39 (PC4); no longer U2.54 (PF7)
- net COL8: now also U2.40 (PC5); no longer U2.51 (PA0)
- net COL9: now also U2.41 (PC6); no longer U2.50 (PA1)
- net CPSLKLED: now also U2.58 (PF3); no longer U2.33 (PE0)
- net D+: now also U3.2 (IO1), USB1.6 (DP1), USB1.8 (DP2)
- net D-: now also U3.3 (IO2), USB1.5 (DN2), USB1.7 (DN1)
- net GND: now also R9.2, C9.2, J2.6 (GND), R8.2, U3.1 (GND), USB1.1 (GND), USB1.12 (GND), USB1.13 (SHIELD)
- net ROW0: now also U2.10 (PB0); no longer U2.17 (PB7)
- net ROW1: now also U2.55 (PF6); no longer U2.38 (PC3)
- net ROW2: now also U2.56 (PF5); no longer U2.39 (PC4)
- net ROW3: now also U2.57 (PF4); no longer U2.40 (PC5)
- net ROW4: now also U2.59 (PF2); no longer U2.41 (PC6)
- net ROW5: now also U2.60 (PF1); no longer U2.42 (PC7)
- net VCC: now also F14.2, U3.4 (VCC), USB1.11 (VBUS), USB1.2 (VBUS); no longer FB1.2
- net RESET: now reaches R2.2, SW1.2, U2.20 (~RESET)
- net RESET: now also J2.5 (~RST)
- net at R9.1: now also USB1.4 (CC1)
- new net: F14.1, FB1.2
- new net: R8.1, USB1.10 (CC2)
- new net MISO: J2.1 (MISO), U2.50 (PA1)
- new net MOSI: J2.4 (MOSI), U2.49 (PA2)
- new net SCK: J2.3 (SCK), U2.51 (PA0)
- no-connect marks 0 -> 2
Other:
- moved on the sheet: C4, C5, C6, C7, LED_CPSLK1, LED_NUMLK1, R_CPSLK1, R_NUMLK1
