File: pcb/pcb.kicad_pcb (KiCad board)
At the start: 2 copper layers, 431.8 x 127 mm, 226 parts, among them J1 MX-NoLED, K0 MX-NoLED, K1 MX-NoLED, K10 MX-NoLED, K2 MX-NoLED, K3 MX-NoLED, K4 MX-NoLED, K5 MX-NoLED, K6 MX-NoLED, K7 MX-NoLED, K8 MX-NoLED, K9 MX-NoLED, M1 MX-NoLED, P1 MX-NoLED, Q1 MX-NoLED, SW1 SW_Push, T1 MX-NoLED, U1 MX-NoLED, U2 AT90USB1286-AU, X1 MX-NoLED, Y1 MX-NoLED, Y2 16 MHz

Commit message: pcb: improve board design
Parts:
- removed F14: 500mA, Fuse:Fuse_1206_3216Metric
- added FB1: Ferrite_Bead_Small, Resistor_SMD:R_0805_2012Metric, B.Cu at (-26.5, 36.1)
- added LED_CPSLK1: LED_Small, LED_SMD:LED_0805_2012Metric, F.Cu at (-35.4, 112.3)
- added LED_NUMLK1: LED_Small, LED_SMD:LED_0805_2012Metric, F.Cu at (310.0, 74.2)
- added R10: 10K, Resistor_SMD:R_0805_2012Metric, F.Cu at (341.4, 38.1)
- added R11: 10K, Resistor_SMD:R_0805_2012Metric, F.Cu at (354.2, 51.1)
- added R12: 10K, Resistor_SMD:R_0805_2012Metric, F.Cu at (358.6, 51.1)
- added R13: 10K, Resistor_SMD:R_0805_2012Metric, F.Cu at (373.4, 49.4)
- added R7: 10K, Resistor_SMD:R_0805_2012Metric, F.Cu at (376.9, 30.9)
- added R9: 10K, Resistor_SMD:R_0805_2012Metric, F.Cu at (376.9, 33.9)
- added R_CPSLK1: 90, Resistor_SMD:R_0805_2012Metric, B.Cu at (-27.9, 112.3)
- added R_NUMLK1: 90, Resistor_SMD:R_0805_2012Metric, B.Cu at (302.5, 74.2)
- added U3: EMI2121MTTAG, Package_DFN_QFN:WDFN-8-1EP_2x2.2mm_P0.5mm_EP0.80x0.54, B.Cu at (-16.8, 30.0)
- BKSP1, ENTER1, NP-0, NP-ENTER1, NP-PLUS1: footprint MX_Alps_Hybrid:MX-1U-NoLED -> MX_Alps_Hybrid:MX-2U-NoLED
- MX-RSHIFT1: footprint MX_Alps_Hybrid:MX-1U-NoLED -> MX_Alps_Hybrid:MX-2.75U-NoLED
- SPACE1: footprint MX_Alps_Hybrid:MX-1U-NoLED -> MX_Alps_Hybrid:MX-6.25U-NoLED
- moved D51 23.1 mm to (208.2, 88.9), turned to 0 degrees
- moved D58 18.1 mm to (358.4, 90.3)
- moved D93 17.8 mm to (358.4, 128.3)
- moved R4 7.92 mm to (-15.9, 37.6)
- moved D30 4.28 mm to (221.9, 56.5), turned to 180 degrees
- moved R3 3.58 mm to (-18.4, 37.6)
- moved D105 0.23 mm to (327.9, 133.7)
- moved NP-ENTER1 0.10 mm to (367.0, 132.5), turned to 90 degrees
- moved NUMLK1 0.07 mm to (309.9, 65.9)
- moved SCLLK1 0.07 mm to (267.0, 37.3)
- moved NP-PLUS1 0.06 mm to (367.0, 94.5), turned to 90 degrees
- turned ENTER1 to 90 degrees
Connections:
- U2 pad 32: Net-(U2-Pad32) -> NUMLKLED
- U2 pad 33: Net-(U2-Pad33) -> CPSLKLED
- USB1 pad 3: D+ -> Net-(U3-Pad1)
- USB1 pad 4: D- -> Net-(U3-Pad2)
- USB1 pad 6: Net-(USB1-Pad6) -> GND
Routing:
- net CPSLKLED: track 0.00 -> 470.2 mm, vias 0 -> 3
- net GND: track 425.1 -> 819.3 mm, vias 0 -> 4
- net +5V: track 409.4 -> 523.6 mm, vias 4 -> 8
- net NUMLKLED: track 0.00 -> 57.2 mm, vias 0 -> 1
- net ROW0: track 480.5 -> 448.0 mm
- net ROW4: track 633.4 -> 611.6 mm
- net VCC: track 5.85 -> 26.8 mm, vias 0 -> 2
- net ROW2: track 614.6 -> 594.8 mm
- net Net-(U3-Pad2): track 0.00 -> 8.55 mm
- net COL21: track 135.7 -> 143.6 mm
- net Net-(U3-Pad1): track 0.00 -> 7.55 mm
- net COL14: track 221.0 -> 215.1 mm
- net COL18: track 128.4 -> 134.2 mm
- net Net-(LED_NUMLK1-Pad2): track 0.00 -> 5.64 mm, vias 0 -> 1
- net Net-(LED_CPSLK1-Pad2): track 0.00 -> 5.64 mm, vias 0 -> 1
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- removed copper zone on B.Cu, net GND

Commit message: pcb: change to usb-c, reorganise pcb
Parts:
- removed R10, R11, R12, R13, R7: 10K, Resistor_SMD:R_0805_2012Metric
- added C9: 0.1uF, Capacitor_SMD:C_0805_2012Metric, B.Cu at (422.7, 27.8)
- added F14: 500mA, Fuse:Fuse_0805_2012Metric, B.Cu at (415.0, 18.2)
- added J2: AVR-ISP-6, random-keyboard-parts:Reset_Pretty-Mask, F.Cu at (394.1, 38.1)
- added R8: 5.1k, Resistor_SMD:R_0805_2012Metric, B.Cu at (427.4, 16.0)
- A1: value MX-NoLED -> A
- ALT1, RALT1: value MX-NoLED -> Alt
- AT1: value MX-NoLED -> @
- B1: value MX-NoLED -> B
- BKSP1: value MX-NoLED -> Backspace
- BSLSH1: value MX-NoLED -> \
- C1: value MX-NoLED -> C
- CAPSL1: value MX-NoLED -> Caps Lock
- COLON1: value MX-NoLED -> :
- COMMA1: value MX-NoLED -> ,
- CTRL1, RCTRL1: value MX-NoLED -> Ctrl
- D59: value MX-NoLED -> D
- DARROW1: value MX-NoLED -> Down
- DASH1, NP-MINUS1: value MX-NoLED -> -
- DEL1, NP-DEL1: value MX-NoLED -> Del
- E1: value MX-NoLED -> E
- END1: value MX-NoLED -> End
- ENTER1, NP-ENTER1: value MX-NoLED -> Enter
- EQUALS1: value MX-NoLED -> =
- ESC1: value MX-NoLED -> Esc
- F1: value MX-NoLED -> F1
- F10: value MX-NoLED -> F10
- F11: value MX-NoLED -> F11
- F12: value MX-NoLED -> F12
- F13: value MX-NoLED -> F
- F2: value MX-NoLED -> F2
- F3: value MX-NoLED -> F3
- F4: value MX-NoLED -> F4
- F5: value MX-NoLED -> F5
- F6: value MX-NoLED -> F6
- F7: value MX-NoLED -> F7
- F8: value MX-NoLED -> F8
- F9: value MX-NoLED -> F9
- FB1: value Ferrite_Bead_Small -> 500mA
- FSLSH1, NP-DIV1: value MX-NoLED -> /
- G1: value MX-NoLED -> G
- H1: value MX-NoLED -> H
- HASH1: value MX-NoLED -> #
- HOME1: value MX-NoLED -> Home
- I1: value MX-NoLED -> I
- INS1: value MX-NoLED -> Insert
- J1: value MX-NoLED -> J
- K0, NP-0: value MX-NoLED -> 0
- K1, NP-1: value MX-NoLED -> 1
- K10: value MX-NoLED -> K
- K2, NP-2: value MX-NoLED -> 2
- K3, NP-3: value MX-NoLED -> 3
- K4, NP-4: value MX-NoLED -> 4
- K5, NP-5: value MX-NoLED -> 5
- K6, NP-6: value MX-NoLED -> 6
- K7, NP-7: value MX-NoLED -> 7
- K8, NP-8: value MX-NoLED -> 8
- K9, NP-9: value MX-NoLED -> 9
- L1: value MX-NoLED -> L
- LARROW1: value MX-NoLED -> Left
- LCBR1: value MX-NoLED -> {
- M1: value MX-NoLED -> M
- MENU1: value MX-NoLED -> Menu
- MX-RSHIFT1, SHIFT1: value MX-NoLED -> Shift
- N1: value MX-NoLED -> N
- NP-MTPLY1: value MX-NoLED -> *
- NP-PLUS1: value MX-NoLED -> +
- NUMLK1: value MX-NoLED -> Num Lock
- O1: value MX-NoLED -> O
- P1: value MX-NoLED -> P
- PAUSE1: value MX-NoLED -> Pause
- PERIOD1: value MX-NoLED -> .
- PGDN1: value MX-NoLED -> Page Down
- PGUP1: value MX-NoLED -> Page Up
- PRTSC1: value MX-NoLED -> Print Screen
- Q1: value MX-NoLED -> Q
- R1: value MX-NoLED -> R
- R9: value 10K -> 5.1k; moved to B.Cu
- RARROW1: value MX-NoLED -> Right
- RCBR1: value MX-NoLED -> }
- S1: value MX-NoLED -> S
- SCLLK1: value MX-NoLED -> Scroll Lock
- SPACE1: value MX-NoLED -> Space
- T1: value MX-NoLED -> T
- TAB1: value MX-NoLED -> Tab
- TILDA1: value MX-NoLED -> ~
- U1: value MX-NoLED -> U
- U3: value EMI2121MTTAG -> PRTR5V0U2X; footprint Package_DFN_QFN:WDFN-8-1EP_2x2.2mm_P0.5mm_EP0.80x0.54 -> random-keyboard-parts:SOT143B
- UARROW1: value MX-NoLED -> Up
- USB1: value Molex-0548190589 -> HRO-TYPE-C-31-M-12; footprint random-keyboard-parts:Molex-0548190589 -> Type-C:HRO-TYPE-C-31-M-12
- V1: value MX-NoLED -> V
- W1: value MX-NoLED -> W
- WIN1, WIN2: value MX-NoLED -> Win
- X1: value MX-NoLED -> X
- Y1: value MX-NoLED -> Y
- Z1: value MX-NoLED -> Z
- moved USB1 443.5 mm to (420.1, 8.26), turned to 0 degrees
- moved FB1 438.1 mm to (411.2, 18.2), turned to 0 degrees
- moved R3 437.7 mm to (419.1, 24.5), turned to 45 degrees
- moved U3 437.0 mm to (420.1, 19.8), turned to 180 degrees
- moved CAPSL1 436.3 mm to (400.6, 91.4)
- moved COLON1 436.3 mm to (598.2, 91.4)
- moved D105 436.3 mm to (764.0, 121.2)
- moved D12 436.3 mm to (649.5, 21.3)
- moved D15 436.3 mm to (711.2, 21.3)
- moved D25 436.3 mm to (554.3, 49.8)
- moved D27 436.3 mm to (592.5, 49.9)
- moved D33 436.3 mm to (730.2, 49.9)
- moved D35 436.3 mm to (773.5, 49.9)
- moved D43 436.3 mm to (506.6, 68.9)
- moved D44 436.3 mm to (525.6, 69.0)
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Connections:
- net Net-(R2-Pad2) renamed RESET
- FB1 pad 2: VCC -> Net-(F14-Pad1)
- R9 pad 2: +5V -> GND
- U2 pad 10: COL16 -> ROW0
- U2 pad 11: COL15 -> Net-(U2-Pad11)
- U2 pad 12: COL14 -> Net-(U2-Pad12)
- U2 pad 13: COL13 -> Net-(U2-Pad13)
- U2 pad 14: COL12 -> Net-(U2-Pad14)
- U2 pad 15: COL11 -> COL15
- U2 pad 16: Net-(U2-Pad16) -> COL16
- U2 pad 17: ROW0 -> COL17
- U2 pad 28: Net-(U2-Pad28) -> COL21
- U2 pad 29: Net-(U2-Pad29) -> COL20
- U2 pad 30: Net-(U2-Pad30) -> COL19
- U2 pad 31: Net-(U2-Pad31) -> COL18
- U2 pad 33: CPSLKLED -> COL1
- U2 pad 34: COL21 -> COL2
- U2 pad 35: COL20 -> COL3
- U2 pad 36: COL19 -> COL4
- U2 pad 37: COL18 -> COL5
- U2 pad 38: ROW1 -> COL6
- U2 pad 39: ROW2 -> COL7
- U2 pad 40: ROW3 -> COL8
- U2 pad 41: ROW4 -> COL9
- U2 pad 42: ROW5 -> COL10
- U2 pad 45: Net-(U2-Pad45) -> COL11
- U2 pad 46: Net-(U2-Pad46) -> COL12
- U2 pad 47: Net-(U2-Pad47) -> COL13
- U2 pad 48: Net-(U2-Pad48) -> COL14
- U2 pad 49: COL10 -> MOSI
- U2 pad 50: COL9 -> MISO
- U2 pad 51: COL8 -> SCK
- U2 pad 54: COL7 -> Net-(U2-Pad54)
- U2 pad 55: COL6 -> ROW1
- U2 pad 56: COL5 -> ROW2
- U2 pad 57: COL4 -> ROW3
- U2 pad 58: COL3 -> CPSLKLED
- U2 pad 59: COL2 -> ROW4
- U2 pad 60: COL1 -> ROW5
- U2 pad 9: COL17 -> Net-(U2-Pad9)
- U3 pad 1: Net-(U3-Pad1) -> GND
- U3 pad 2: Net-(U3-Pad2) -> D+
- U3 pad 3: GND -> D-
- U3 pad 4: GND -> VCC
- USB1 pad 2: Net-(USB1-Pad2) -> VCC
- USB1 pad 3: Net-(U3-Pad1) -> Net-(USB1-Pad3)
- USB1 pad 4: Net-(U3-Pad2) -> Net-(R9-Pad1)
- USB1 pad 5: VCC -> D-
- USB1 pad 6: GND -> D+
Routing:
- net GND: track 819.3 -> 155.5 mm
- net CPSLKLED: track 470.2 -> 109.5 mm, vias 3 -> 1
- net COL20: track 118.6 -> 459.3 mm
- net COL1: track 427.4 -> 88.1 mm, vias 0 -> 1
- net COL21: track 143.6 -> 482.6 mm
- net COL0: track 476.7 -> 139.2 mm
- net Net-(R4-Pad1): track 333.5 -> 2.80 mm, vias 2 -> 0
- net Net-(R3-Pad1): track 332.9 -> 2.92 mm
- net COL19: track 92.3 -> 416.7 mm
- net NUMLKLED: track 57.2 -> 359.7 mm
- net COL2: track 427.1 -> 134.9 mm, vias 0 -> 1
- net COL18: track 134.2 -> 423.1 mm
- net COL17: track 134.9 -> 407.1 mm
- net COL3: track 433.2 -> 180.0 mm, vias 0 -> 1
- net COL16: track 164.7 -> 386.4 mm
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- added copper zone on B.Cu, net GND
- added copper zone on F.Cu, net GND
Other:
- board size 431.8 x 127 mm -> 431.8 x 130.9 mm

Commit message: pcb: update edge cuts
Parts:
- moved D15 434.3 mm to (277.1, 33.3)
- moved D54 434.3 mm to (296.4, 80.9)
- moved D67 434.3 mm to (115.3, 99.9)
- moved D71 434.3 mm to (191.6, 99.9)
- moved NP-0 434.3 mm to (321.4, 141.4)
- moved NP-ENTER1 434.3 mm to (369.0, 131.8)
- moved NP-MINUS1 434.3 mm to (369.0, 65.2)
- moved NUMLK1 434.3 mm to (311.9, 65.3)
- moved PAUSE1 434.3 mm to (288.1, 36.7)
- moved PGDN1 434.3 mm to (288.1, 84.3)
- moved PGUP1 434.3 mm to (288.1, 65.2)
- moved RARROW1 434.3 mm to (288.1, 141.4)
- moved A1 434.3 mm to (-7.30, 103.3)
- moved ALT1 434.3 mm to (9.46, 141.4)
- moved AT1 434.3 mm to (183.2, 103.3)
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Other:
- outline, holes or cut-outs redrawn
